File: microcontroller.kicad_sch (KiCad schematic)
At the start: 7 parts, among them U1 EFM8BB10F8G-A-SOIC16

Commit message: Created new hierarchy, added new nRF MCU, started really digging into schematic
Parts:
- removed U1: EFM8BB10F8G-A-SOIC16, Package_SO:SOIC-16_3.9x9.9mm_P1.27mm, symbol MCU_SiliconLabs:EFM8BB10F8G-A-SOIC16
- added C3, C4, C5, C6: 100n, symbol Device:C_Small
- added U1: NRF54L15-QFAA-R, Team_512_MCUs:NRF54L15-QFAA-R, symbol Team_512_MCUs:NRF54L15-QFAA-R
- C2: value 10n -> 100n
Connections:
- net +3.3V: no longer C1.1, C2.1
- net GND: now also C3.2, C4.2, C5.2, C6.2, U1.32 (VSS_PA), U1.44 (VSS), U1.49 (VSS)
- net C2CK renamed SWDCLK
- net SWDCLK: now also U1.26 (SWDCLK)
- net C2D renamed SWDIO
- net SWDIO: now also U1.25 (SWDIO)
- new net 3V3: C1.1, C2.1, C3.1, C4.1, C5.1, C6.1, U1.10 (VDD), U1.22 (VDD), U1.36 (VDD), U1.47 (VDD), U1.48 (VDD)
Other:
- moved on the sheet: C1, C2, TP1, TP2, TP3, TP4
