File: FT2232.kicad_sch (KiCad schematic)
At the start: 38 parts, among them J1 2.54mm, Q1 SMMBT3904LT1G, Q2 SMMBT3904LT1G, Q3 SMMBT3904LT1G, Q4 SMMBT3904LT1G, U4 FT2232HL, Y1 ABM8AIG-12.000MHZ-12-2Z-T3

Commit message: Finished schematic, added power section for external power (both power supply and battery), added current sensing for TX microcontroller
Parts:
- renumbered C12 to C32, C13 to C33, C14 to C34, C15 to C35, C16 to C36, C17 to C37, C18 to C38, C19 to C39, C20 to C40, C21 to C41, C22 to C42, C23 to C43, C24 to C44, C25 to C45, C26 to C46, R4 to R17, R5 to R18, R6 to R19, R7 to R20, R8 to R21, R9 to R22, R10 to R23, R11 to R24, R12 to R25, R13 to R26, R14 to R27, R15 to R28, U4 to U7, Y1 to Y3

Commit message: Made most capacitors 0402 for mcu sheets, defined board shape and started layout
Parts:
- removed C33, C34: 4.7u, Capacitor_SMD:C_0603_1608Metric, symbol Device:C_Small
- removed C35, C36, C37, C40, C41, C42, C43, C44, C45, C46: 100n, Capacitor_SMD:C_0603_1608Metric, symbol Device:C_Small
- removed C39: 3.3u, Capacitor_SMD:C_0603_1608Metric, symbol Device:C_Small
- added C35, C36: 4.7u, Capacitor_SMD:C_0603_1608Metric_Pad1.08x0.95mm_HandSolder, symbol AERO_Capacitors:C_0603
- added C37, C38, C39, C42, C43, C44, C45, C46, C47, C48: 100n, Capacitor_SMD:C_0603_1608Metric_Pad1.08x0.95mm_HandSolder, symbol AERO_Capacitors:C_0603
- added C41: 3.3u, Capacitor_SMD:C_0603_1608Metric_Pad1.08x0.95mm_HandSolder, symbol AERO_Capacitors:C_0603
- renumbered C32 to C34, C38 to C40, J1 to J2, R17 to R18, R18 to R19, R19 to R20, R20 to R21, R21 to R22, R22 to R23, R23 to R24, R24 to R25, R25 to R26, R26 to R27, R27 to R28, R28 to R29
Connections:
- net 1V8: now also C41.1, C42.1, C43.1, C45.1
- net 3V3: now also C38.1, C44.1, C46.1, C47.1, C48.1
- net GND: now also C35.2, C36.2, C37.2, C38.2, C39.2, C41.2, C42.2, C43.2, C44.2, C45.2, C46.2, C47.2, C48.2
- net at R19.2, U7.4 (VPHY): now also C36.1, C39.1
- net at R18.2, U7.9 (VPLL): now also C35.1, C37.1
