File: piezo_TX.kicad_sch (KiCad schematic)
At the start: 5 parts, among them J4 1053091102

Commit message: Made most capacitors 0402 for mcu sheets, defined board shape and started layout
Parts:
- renumbered C52 to C17, C53 to C18, J4 to J1, R11 to R12, R12 to R13
Changed lines of the file:
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@@
 		(dnp no)
 		(fields_autoplaced yes)
-		(property "Reference" "#PWR062"
+		(property "Reference" "#PWR022"
 			(at 151.13 100.33 0)
 			(hide yes)
@@
 			(project "Temp-Logger"
 				(path "/9c5f4d5b-9930-4cae-a7d7-03685cadac72/fcea2aa9-9943-4e17-9260-3f9a95f3f7ce/c3629570-a093-47e6-a19a-b1d25f71c5ae"
-					(reference "#PWR062")
+					(reference "#PWR022")
 					(unit 1)
 				)
@@
 		(in_pos_files yes)
 		(dnp yes)
-		(property "Reference" "C53"
+		(property "Reference" "C18"
 			(at 153.67 112.268 0)
 			(show_name no)
@@
 			(project "Temp-Logger"
 				(path "/9c5f4d5b-9930-4cae-a7d7-03685cadac72/fcea2aa9-9943-4e17-9260-3f9a95f3f7ce/c3629570-a093-47e6-a19a-b1d25f71c5ae"
-					(reference "C53")
+					(reference "C18")
 					(unit 1)
 				)
@@
 		(dnp no)
 		(fields_autoplaced yes)
-		(property "Reference" "R11"
+		(property "Reference" "R12"
 			(at 139.7 77.47 0)
 			(show_name no)
@@
 			(project "Temp-Logger"
 				(path "/9c5f4d5b-9930-4cae-a7d7-03685cadac72/fcea2aa9-9943-4e17-9260-3f9a95f3f7ce/c3629570-a093-47e6-a19a-b1d25f71c5ae"
-					(reference "R11")
+					(reference "R12")
 					(unit 1)
 				)
@@
 		(in_pos_files yes)
 		(dnp yes)
-		(property "Reference" "C52"
+		(property "Reference" "C17"
 			(at 153.67 85.598 0)
 			(show_name no)
@@
 			(project "Temp-Logger"
 				(path "/9c5f4d5b-9930-4cae-a7d7-03685cadac72/fcea2aa9-9943-4e17-9260-3f9a95f3f7ce/c3629570-a093-47e6-a19a-b1d25f71c5ae"
-					(reference "C52")
+					(reference "C17")
 					(unit 1)
 				)
@@
 		(dnp no)
 		(fields_autoplaced yes)
-		(property "Reference" "#PWR063"
+		(property "Reference" "#PWR023"
 			(at 151.13 127 0)
 			(hide yes)
@@
 			(project "Temp-Logger"
 				(path "/9c5f4d5b-9930-4cae-a7d7-03685cadac72/fcea2aa9-9943-4e17-9260-3f9a95f3f7ce/c3629570-a093-47e6-a19a-b1d25f71c5ae"
-					(reference "#PWR063")
+					(reference "#PWR023")
 					(unit 1)
 				)
@@
 		(dnp no)
 		(fields_autoplaced yes)
-		(property "Reference" "R12"
+		(property "Reference" "R13"
 			(at 139.7 104.14 0)
 			(show_name no)
@@
 			(project "Temp-Logger"
 				(path "/9c5f4d5b-9930-4cae-a7d7-03685cadac72/fcea2aa9-9943-4e17-9260-3f9a95f3f7ce/c3629570-a093-47e6-a19a-b1d25f71c5ae"
-					(reference "R12")
+					(reference "R13")
 					(unit 1)
 				)
@@
 		(in_pos_files yes)
 		(dnp no)
-		(property "Reference" "J4"
+		(property "Reference" "J1"
 			(at 189.23 90.17 0)
 			(show_name no)
@@
 			(project "Temp-Logger"
 				(path "/9c5f4d5b-9930-4cae-a7d7-03685cadac72/fcea2aa9-9943-4e17-9260-3f9a95f3f7ce/c3629570-a093-47e6-a19a-b1d25f71c5ae"
-					(reference "J4")
+					(reference "J1")
 					(unit 1)
 				)
