File: tx_microcontroller.kicad_sch (KiCad schematic)
At the start: 13 parts, among them U1 NRF54L15-QFAA-R

Commit message: Added USB to UART circuitry, cleaned up top sheets, added more supporting circuitry for TX MCU
Parts:
- added C10, C7, C8: 2.2u, Capacitor_SMD:C_0603_1608Metric_Pad1.08x0.95mm_HandSolder, symbol AERO_Capacitors:C_0603
- added C6: 3.9p, Capacitor_SMD:C_0603_1608Metric_Pad1.08x0.95mm_HandSolder, symbol AERO_Capacitors:C_0603
- added C9: 10n, Capacitor_SMD:C_0603_1608Metric_Pad1.08x0.95mm_HandSolder, symbol AERO_Capacitors:C_0603
- added L2: 4.7u, Inductor_SMD:L_0603_1608Metric_Pad1.05x0.95mm_HandSolder, symbol Device:L_Small
- added R21: 0, Resistor_SMD:R_0603_1608Metric_Pad0.98x0.95mm_HandSolder, symbol AERO_Resistors:R_0603
- added TP10, TP11, TP12, TP13, TP9: 1.0mm, TestPoint:TestPoint_Pad_D1.0mm, symbol Connector:TestPoint
- R1: renamed from R4; value 4.7k -> 1k
- renumbered C6 to C3, R1 to R2, R2 to R3
Connections:
- net 3V3: now also TP9.1; no longer R1.2
- net GND: now also U1.32 (VSS_PA), C10.2, C6.2, C7.2, C8.2, C9.2
- net at U1.33 (DECRF): now also U1.43 (DECA), C10.1, C8.1, C9.1, R21.1, TP12.1
- net at U1.45 (DECD): now also C7.1, L2.1, R21.2, TP11.1
- net at U1.46 (DCC): now also L2.2, TP10.1
- net BOOT_A: now reaches U1.24 (P0.01)
- net TX+ renamed PWM+
- net TX- renamed PWM-
- net nRF_RXD_A renamed nRF_URXD_A
- net nRF_TXD_A renamed nRF_UTXD_A
- net nRF_~{RST} renamed ~{RESET}
- net ~{RESET}: now also C6.1, TP13.1
- new net nRF_~{RESET}_A: R1.2
Other:
- note added: "Add buttons for reset and boot"
- note added: "Change to header?"
- note added: "Replace w/ FB if needed"
- note added: "~{RESET} pulled up internally"
- moved on the sheet: R1

Commit message: Finished schematic, added power section for external power (both power supply and battery), added current sensing for TX microcontroller
Parts:
- removed C1: 10u, symbol Device:C_Small
- removed C10: 2.2u, Capacitor_SMD:C_0603_1608Metric_Pad1.08x0.95mm_HandSolder, symbol AERO_Capacitors:C_0603
- removed C4, C5: 100n, symbol Device:C_Small
- removed C9: 10n, Capacitor_SMD:C_0603_1608Metric_Pad1.08x0.95mm_HandSolder, symbol AERO_Capacitors:C_0603
- removed R1: 1k, Resistor_SMD:R_0603_1608Metric_Pad0.98x0.95mm_HandSolder, symbol AERO_Resistors:R_0603
- removed R2, R3: 4.7k, Resistor_SMD:R_0603_1608Metric_Pad0.98x0.95mm_HandSolder, symbol AERO_Resistors:R_0603
- removed R21: 0, Resistor_SMD:R_0603_1608Metric_Pad0.98x0.95mm_HandSolder, symbol AERO_Resistors:R_0603
- removed TP10, TP11, TP12, TP13: 1.0mm, TestPoint:TestPoint_Pad_D1.0mm, symbol Connector:TestPoint
- removed unit 1 of U1
- added C1, C5: 2.2u, Capacitor_SMD:C_0603_1608Metric_Pad1.08x0.95mm_HandSolder, symbol AERO_Capacitors:C_0603
- added C10, C11, C14: 100n, symbol Device:C_Small
- added C12: 2.0p, Capacitor_SMD:C_0201_0603Metric, symbol Device:C_Small
- added C13: 8p, Capacitor_SMD:C_0603_1608Metric_Pad1.08x0.95mm_HandSolder, symbol AERO_Capacitors:C_0603
- added C15: 0.3p, Capacitor_SMD:C_0201_0603Metric, symbol Device:C_Small
- added C4: 10n, Capacitor_SMD:C_0603_1608Metric_Pad1.08x0.95mm_HandSolder, symbol AERO_Capacitors:C_0603
- added C9: 1.5p, Capacitor_SMD:C_0201_0603Metric, symbol Device:C_Small
- added L1: 4.7u, Inductor_SMD:L_0603_1608Metric_Pad1.05x0.95mm_HandSolder, symbol Device:L_Small
- added L3, L4: 3.5n, Inductor_SMD:L_0201_0603Metric, symbol Device:L_Small
- added R10, R5, R9: 0, Resistor_SMD:R_0603_1608Metric_Pad0.98x0.95mm_HandSolder, symbol AERO_Resistors:R_0603
- added R38: 100m, Resistor_SMD:R_1206_3216Metric_Pad1.30x1.75mm_HandSolder, symbol AERO_Resistors:R_1206
- added R6: 1k, Resistor_SMD:R_0603_1608Metric_Pad0.98x0.95mm_HandSolder, symbol AERO_Resistors:R_0603
- added R7, R8: 4.7k, Resistor_SMD:R_0603_1608Metric_Pad0.98x0.95mm_HandSolder, symbol AERO_Resistors:R_0603
- added SW1: KMR211G LFS, Button_Switch_SMD:SW_Push_1P1T_NO_CK_KMR2, symbol Switch:SW_Push
- added TP19, TP20, TP5, TP6, TP7, TP8: 1.0mm, TestPoint:TestPoint_Pad_D1.0mm, symbol Connector:TestPoint
- added unit 1 of U1
- added Y1: ECS-320-CDX-2374, Team_512_Oscillators:ECS-320-CDX-2374, symbol Team_512_Oscillators:ECS-320-CDX-2374
- C2: value 100n -> 10u
- C6: value 3.9p -> 2.2u
- C7: value 2.2u -> 8p; Tolerance 20% -> 10%; now not fitted
- C8: value 2.2u -> 3.9p
- L2: value 4.7u -> 2.7n; footprint Inductor_SMD:L_0603_1608Metric_Pad1.05x0.95mm_HandSolder -> Inductor_SMD:L_0201_0603Metric; Part Number (none) -> GJM0335C1E1R5WB01
- U1: value NRF54L15-QFAA-R -> nRF54L15-QFAA-R
Connections:
- net +3.3V: now also TP6.1; no longer TP1.1
- net 3V3: now also R38.1, TP19.1; no longer C2.1, C3.1, TP9.1
- net GND: now also TP9.1, C1.2, C10.2, C11.2, C12.2, C13.2, C14.2, C15.2, C4.2, C5.2, C9.2, SW1.1, U1.32 (VSS_PA), U1.44 (VSS), U1.49 (VSS), Y1.2 (GND), Y1.4 (GND); no longer TP4.1
- net PWM+: now also R9.1; no longer U1.5 (P1.04/AIN0/TAMPC)
- net PWM-: now also R10.1; no longer U1.8 (P1.07/AIN3/TAMPC)
- net SCL: now also R8.1
- net SDA: now also R7.1
- net SWDCLK: now also TP7.1, U1.26 (SWDCLK); no longer TP2.1
- net SWDIO: now also TP8.1, U1.25 (SWDIO); no longer TP3.1
- net nRF_~{RESET}_A: now also R6.2, SW1.2
- net ~{RESET}: now also C8.1, R6.1, TP5.1, U1.30 (~{RESET}); no longer C6.1
- net at L2.1: now also U1.31 (ANT); no longer C7.1
- net at L2.2: now also C9.1, L3.1
- new net: C1.1, C4.1, C5.1, R5.1, TP3.1, U1.33 (DECRF), U1.43 (DECA)
- new net: C12.1, L3.2, L4.1
- new net: L1.2, TP2.1, U1.46 (DCC)
- new net: R9.2, U1.5 (P1.04/AIN0/TAMPC)
- new net: R10.2, U1.8 (P1.07/AIN3/TAMPC)
- new net: C6.1, L1.1, R5.2, TP1.1, U1.45 (DECD)
- new net: C13.1, U1.34 (XC1), Y1.3
- new net: C7.1, U1.35 (XC2), Y1.1
- new net RF: C15.1, L4.2
- new net TX3V3: C10.1, C11.1, C14.1, C2.1, C3.1, R38.2, R7.2, R8.2, TP20.1, TP4.1, U1.10 (VDD), U1.22 (VDD), U1.36 (VDD), U1.47 (VDD), U1.48 (VDD)
- no-connect marks 0 -> 22
Other:
- note added: "ADD OSCILLATOR"
- note added: "Resistor and test points for measuring current draw"
- note added: "SEE DATASHEET FOR GND ROUTING"
- note removed: "Add buttons for reset and boot"

Commit message: Made most capacitors 0402 for mcu sheets, defined board shape and started layout
Parts:
- removed C1, C5, C6: 2.2u, Capacitor_SMD:C_0603_1608Metric_Pad1.08x0.95mm_HandSolder, symbol AERO_Capacitors:C_0603
- removed C10, C11, C14, C3: 100n, symbol Device:C_Small
- removed C2: 10u, symbol Device:C_Small
- removed C4: 10n, Capacitor_SMD:C_0603_1608Metric_Pad1.08x0.95mm_HandSolder, symbol AERO_Capacitors:C_0603
- removed C8: 3.9p, Capacitor_SMD:C_0603_1608Metric_Pad1.08x0.95mm_HandSolder, symbol AERO_Capacitors:C_0603
- removed R5: 0, Resistor_SMD:R_0603_1608Metric_Pad0.98x0.95mm_HandSolder, symbol AERO_Resistors:R_0603
- added C1, C6: 2.2u, Capacitor_SMD:C_0402_1005Metric_Pad0.74x0.62mm_HandSolder, symbol AERO_Capacitors:C_0402
- added C10, C11, C14, C3: 100n, Capacitor_SMD:C_0402_1005Metric_Pad0.74x0.62mm_HandSolder, symbol AERO_Capacitors:C_0402
- added C2: 10u, Capacitor_SMD:C_0402_1005Metric_Pad0.74x0.62mm_HandSolder, symbol AERO_Capacitors:C_0402
- added C4: 10n, Capacitor_SMD:C_0402_1005Metric_Pad0.74x0.62mm_HandSolder, symbol AERO_Capacitors:C_0402
- added C5: 2.2n, Capacitor_SMD:C_0402_1005Metric_Pad0.74x0.62mm_HandSolder, symbol AERO_Capacitors:C_0402
- added C8: 3.9p, Capacitor_SMD:C_0402_1005Metric_Pad0.74x0.62mm_HandSolder, symbol AERO_Capacitors:C_0402
- added R5: 0, Resistor_SMD:R_0402_1005Metric_Pad0.72x0.64mm_HandSolder, symbol AERO_Resistors:R_0402
- renumbered R9 to R10, R10 to R11, R38 to R6, R6 to R7, R7 to R8, R8 to R9, TP8 to TP10, TP9 to TP11, TP19 to TP2, TP2 to TP3, TP3 to TP4, TP20 to TP5, TP4 to TP6, TP5 to TP7, TP6 to TP8, TP7 to TP9
Connections:
- net +3.3V is gone; now on net TX3V3: TP8.1
- net GND: now also C1.2, C10.2, C11.2, C14.2, C2.2, C3.2, C4.2, C5.2, C6.2, C8.2
- net TX3V3: now also C10.1, C11.1, C14.1, C2.1, C3.1
- net ~{RESET}: now also C8.1
- net at TP4.1, U1.33 (DECRF), U1.43 (DECA): now also C1.1, C4.1, C5.1, R5.2
- net at L1.1, TP1.1, U1.45 (DECD): now also C6.1, R5.1
